File: EV-Front-SDC/EV-Front-SDC.kicad_pcb (KiCad board)
At the start: 2 copper layers, 78 x 58 mm, 28 parts, among them J1 JST-XA, J2 GPS, J2 JST-XA, J3 IMU, J3 JST-XA, J4 JST-XA, J5 JST-XA, J8 Conn_01x14, Q1 BSS205N, Q2 BSS205N, Q3 BSS205N, U2 MCP23S08-E_SS

Commit message: Routed the PCB
Parts:
- removed C1: 1u, Capacitor_SMD:C_0603_1608Metric
- removed the J2 at (186.8, 67.8)
- removed the J3 at (176.3, 67.9)
- removed J4, J5: JST-XA, Custom_MSM:Connector_JST-XA_2POS
- removed J8: Conn_01x14, Connector_JST:JST_XA_S14B-XASK-1_1x14_P2.50mm_Horizontal
- removed R10: 10k, Resistor_SMD:R_0603_1608Metric
- added C11: 0.1u, Capacitor_SMD:C_0805_2012Metric, F.Cu at (86.9, 106.4)
- added C12: 0.1u, Capacitor_SMD:C_0805_2012Metric, F.Cu at (86.7, 102.9)
- added C13: 1u, Capacitor_SMD:C_0805_2012Metric, F.Cu at (90.5, 102.9)
- added C3: 0.1u, Capacitor_SMD:C_0805_2012Metric, F.Cu at (84.3, 92.7)
- added C4: 10u, Capacitor_SMD:C_0805_2012Metric, F.Cu at (73.5, 117.9)
- added C5: 1u, Capacitor_SMD:C_0805_2012Metric, F.Cu at (93.5, 118.8)
- added C6: 1u, Capacitor_SMD:C_0805_2012Metric, F.Cu at (73.5, 115.8)
- added C7: 0.1u, Capacitor_SMD:C_0805_2012Metric, F.Cu at (73.5, 112.3)
- added R11: 10k, Resistor_SMD:R_0805_2012Metric, F.Cu at (84.3, 98.6)
- added R12: 10k, Resistor_SMD:R_0805_2012Metric, F.Cu at (84.3, 95.5)
- added U1: TXE8116DGSR, Package_DFN_QFN:QFN-24-1EP_4x4mm_P0.5mm_EP2.7x2.7mm, F.Cu at (78.4, 95.0)
- added U3: MAX3390EEUD_T, Custom_MSM:SOP65P640X110-14N, F.Cu at (80.7, 104.8)
- C2: footprint Capacitor_SMD:C_0603_1608Metric -> Capacitor_SMD:C_0805_2012Metric
- D1, D2, D3: footprint LED_SMD:LED_0603_1608Metric -> LED_SMD:LED_0805_2012Metric
- J1: value JST-XA -> B06B-PASK_LF__SN_; footprint Custom_MSM:Connector_JST-XA_2POS -> Custom_MSM:S06BXASK1LFSN
- J3: value IMU -> Conn_01x14; footprint CustomFootprints10:IMU -> Connector_JST:JST_XA_S14B-XASK-1_1x14_P2.50mm_Horizontal
- R1, R2, R3: value 40k -> 75K; footprint Resistor_SMD:R_0603_1608Metric -> Resistor_SMD:R_0805_2012Metric
- R4, R5, R6: footprint Resistor_SMD:R_0603_1608Metric -> Resistor_SMD:R_0805_2012Metric
- R7, R8, R9: value 10k -> 25k; footprint Resistor_SMD:R_0603_1608Metric -> Resistor_SMD:R_0805_2012Metric
- U2: value MCP23S08-E_SS -> SCH16T-K01-10; footprint Custom_MSM:SOP65P780X200-20N -> Custom_MSM:SCH16TK0110
- moved J1 149.9 mm to (54.1, 112.6)
- moved J2 118.2 mm to (75.3, 80.5)
- moved R1 110.9 mm to (52.6, 106.0), turned to -90 degrees
- moved R7 107.0 mm to (52.5, 101.3), turned to -90 degrees
- moved Q1 104.1 mm to (56.8, 103.6), turned to 90 degrees
- moved R2 102.1 mm to (60.9, 106.2), turned to -90 degrees
- moved D1 98.3 mm to (56.7, 96.6), turned to 90 degrees
- moved R8 97.5 mm to (60.9, 101.2), turned to -90 degrees
- moved R3 95.9 mm to (67.7, 106.4), turned to -90 degrees
- moved Q2 95.6 mm to (64.8, 103.7), turned to 90 degrees
- moved R4 95.1 mm to (56.7, 92.8), turned to -90 degrees
- moved REF** 91.4 mm to (81.2, 93.2)
- moved R9 90.8 mm to (67.8, 101.4), turned to -90 degrees
- moved D2 89.3 mm to (64.6, 96.5), turned to 90 degrees
- moved J3 89.2 mm to (100.0, 110.3), turned to 90 degrees
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Connections:
- C2 pad 1: +5V -> +3V3
- J1 pad 1: Net-(J1-Pin_1) -> Rear_SDC_In(Right)
- J3 pad 1: +3V3 -> 5V_CS_C
- J3 pad 10: unconnected-(J3-Pin_10-Pad10) -> TX
- J3 pad 2: unconnected-(J3-Pin_2-Pad2) -> 5V_CS_D
- J3 pad 3: GND -> 5V_SCLK
- J3 pad 4: SCL -> 5V_MISO
- J3 pad 5: SDA -> 5V_MOSI
- J3 pad 6: unconnected-(J3-Pin_6-Pad6) -> PPS
- J3 pad 9: unconnected-(J3-Pin_9-Pad9) -> RX
- U2 pad 1: 5V_SCLK -> GND
- U2 pad 10: unconnected-(U2-NC-Pad10) -> Net-(U2-VREGA)
- U2 pad 11: unconnected-(U2-NC-Pad10)_1 -> Net-(U2-VREGA)
- U2 pad 12: BOTS_S -> GND
- U2 pad 13: CK_S -> GND
- U2 pad 14: IS_S -> Net-(U2-VREGD)
- U2 pad 15: unconnected-(U2-GP3-Pad15) -> Net-(U2-VREGD)
- U2 pad 16: unconnected-(U2-GP4-Pad16) -> GND
- U2 pad 17: unconnected-(U2-GP5-Pad17) -> +3V3
- U2 pad 18: unconnected-(U2-GP6-Pad18) -> +3V3
- U2 pad 19: unconnected-(U2-GP7-Pad19) -> MISO
- U2 pad 2: 5V_MOSI -> unconnected-(U2-N.C.-Pad2)
- U2 pad 20: +5V -> unconnected-(U2-DRY_SYNC-Pad20)
- U2 pad 3: 5V_MISO -> unconnected-(U2-TA9-Pad3)
- U2 pad 4: +5V -> unconnected-(U2-TA8-Pad4)
- U2 pad 6: Net-(U2-~{RESET}) -> unconnected-(U2-EXTRESN-Pad6)
- U2 pad 7: 5V_CS_C -> GND
- U2 pad 8: unconnected-(U2-INT-Pad8) -> +3V3
Routing:
- net +3V3: track 0.00 -> 108.0 mm
- net +5V: track 4.95 -> 92.3 mm, vias 0 -> 1
- net PPS: track 0.00 -> 50.9 mm
- net BOTS_S: track 0.00 -> 44.8 mm, vias 0 -> 2
- net 5V_MISO: track 0.00 -> 40.1 mm, vias 0 -> 1
- net GND: track 0.00 -> 37.5 mm, vias 0 -> 13
- net 5V_CS_C: track 0.00 -> 28.7 mm, vias 0 -> 1
- net 5V_MOSI: track 0.00 -> 28.0 mm
- net 5V_SCLK: track 0.00 -> 27.9 mm
- net CK_S: track 0.00 -> 24.0 mm
- net RX: track 0.00 -> 24.0 mm
- net MISO: track 0.00 -> 22.8 mm
- net CS_D: track 0.00 -> 18.4 mm, vias 0 -> 2
- net TX: track 0.00 -> 17.7 mm
- net 5V_CS_D: track 0.00 -> 17.5 mm
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- added copper zone on B.Cu, net GND
- added copper zone on F.Cu, net GND
Other:
- outline, holes or cut-outs redrawn

Commit message: Fixed GPIO footprint + added signature
Parts:
- added G***: LOGO, LOGO, F.Cu at (47.0, 81.0)
- U1: value TXE8116DGSR -> ~
- moved U1 0.45 mm to (78.0, 95.0), turned to 0 degrees
Connections:
- C12 pad 2: Net-(C12-Pad2) -> GND
- C13 pad 2: Net-(C12-Pad2) -> GND
- R11 pad 1: Net-(U1-~{RESET}) -> Net-(U1-RESET)
- R12 pad 1: Net-(U1-~{INT}) -> Net-(U1-INT)
- U1 pad 1: Net-(U1-~{INT}) -> unconnected-(U1-P0.5-Pad1)
- U1 pad 12: unconnected-(U1-P0.7-Pad12) -> 5V_CS_C
- U1 pad 13: unconnected-(U1-P1.7-Pad13) -> 5V_SCLK
- U1 pad 14: unconnected-(U1-P1.6-Pad14) -> 5V_MOSI
- U1 pad 15: unconnected-(U1-P1.5-Pad15) -> Net-(U1-RESET)
- U1 pad 16: unconnected-(U1-P1.4-Pad16) -> Net-(U1-INT)
- U1 pad 17: unconnected-(U1-P1.3-Pad17) -> 5V_MISO
- U1 pad 18: unconnected-(U1-P1.2-Pad18) -> +5V
- U1 pad 19: unconnected-(U1-P1.1-Pad19) -> GND
- U1 pad 2: 5V_MISO -> unconnected-(U1-P0.6-Pad2)
- U1 pad 20: unconnected-(U1-P1.0-Pad20) -> BOTS_S
- U1 pad 21: 5V_CS_C -> CK_S
- U1 pad 22: 5V_SCLK -> IS_S
- U1 pad 23: 5V_MOSI -> unconnected-(U1-P0.3-Pad23)
- U1 pad 24: Net-(U1-~{RESET}) -> unconnected-(U1-P0.4-Pad24)
- U1 pad 3: +5V -> unconnected-(U1-P0.7-Pad3)
- U1 pad 4: GND -> unconnected-(U1-P1.7-Pad4)
- U1 pad 5: BOTS_S -> unconnected-(U1-P1.6-Pad5)
- U1 pad 6: CK_S -> unconnected-(U1-P1.5-Pad6)
- U1 pad 7: IS_S -> unconnected-(U1-P1.4-Pad7)
Routing:
- net BOTS_S: track 44.8 -> 30.2 mm
- net GND: track 37.5 -> 47.8 mm
- net 5V_MISO: track 40.1 -> 32.5 mm, vias 1 -> 2
- net Net-(U1-RESET): track 0.00 -> 5.29 mm
- net Net-(C12-Pad2): track 4.61 -> 0.00 mm
- net Net-(U1-~{RESET}): track 4.41 -> 0.00 mm
- net Net-(U1-INT): track 0.00 -> 3.74 mm
- net Net-(U1-~{INT}): track 3.35 -> 0.00 mm
- net CK_S: track 24.0 -> 21.5 mm
- net 5V_MOSI: track 28.0 -> 29.4 mm, vias 0 -> 1
- net IS_S: track 14.9 -> 13.6 mm
- net +5V: track 92.3 -> 91.7 mm

Commit message: Re-routed and bomed
Parts:
- removed the G*** at (47.0, 81.0)
- added G***: LOGO, LOGO, F.Cu at (103.0, 117.1)
- added G***: LOGO, LOGO, B.Cu at (70.0, 84.0)
- added REF**: LOGO, Custom_MSM:Decorative_Stinger, F.Cu at (98.8, 69.6)
- J1: value B06B-PASK_LF__SN_ -> Conn_01x06; footprint Custom_MSM:S06BXASK1LFSN -> Connector_JST:JST_XA_S06B-XASK-1_1x06_P2.50mm_Horizontal
- Q1, Q2, Q3, R1, R2, R3, R7, R8, R9: moved to B.Cu
- R4, R5, R6: value 300 -> 300R
- moved R6 14.7 mm to (60.8, 102.2)
- moved D3 14.7 mm to (60.8, 106.2)
- moved D2 13.4 mm to (55.0, 105.9)
- moved R5 13.4 mm to (55.0, 102.1)
- moved D1 12.3 mm to (48.9, 106.1)
- moved R4 12.3 mm to (48.9, 102.4)
- moved U3 10.4 mm to (91.0, 106.2)
- moved C3 10.3 mm to (93.0, 98.2), turned to 180 degrees
- moved Q1 8.59 mm to (48.2, 104.0)
- moved Q2 8.28 mm to (56.5, 104.0)
- moved Q3 7.50 mm to (64.5, 104.0)
- moved C11 7.44 mm to (93.2, 110.2), turned to 180 degrees
- moved C12 6.90 mm to (93.0, 100.2), turned to 180 degrees
- moved U1 5.51 mm to (77.3, 100.4)
- moved J2 4.28 mm to (71.1, 80.1)
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Routing:
- net +3V3: track 108.0 -> 161.9 mm, vias 0 -> 2
- net GND: track 47.8 -> 0.00 mm, vias 13 -> 3
- net 5V_CS_C: track 29.2 -> 58.6 mm, vias 1 -> 0
- net +5V: track 91.7 -> 79.4 mm, vias 1 -> 2
- net BOTS_S: track 30.2 -> 41.4 mm, vias 2 -> 1
- net 5V_CS_D: track 17.5 -> 6.54 mm
- net CK_S: track 21.5 -> 30.3 mm, vias 0 -> 1
- net CS_D: track 18.4 -> 10.3 mm
- net IS_S: track 13.6 -> 21.4 mm, vias 0 -> 1
- net 5V_MISO: track 32.5 -> 25.3 mm
- net MISO: track 22.8 -> 17.2 mm
- net 5V_SCLK: track 27.9 -> 23.0 mm, vias 0 -> 2
- net 5V_MOSI: track 29.4 -> 24.8 mm, vias 1 -> 0
- net TX: track 17.7 -> 22.2 mm
- net MOSI: track 15.6 -> 11.4 mm
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Other:
- board text added: "BOTS"
- board text added: "CK"
- board text added: "Front SDC V1.0 Designed by Ahmed Kandil Routed 26/10/2026"
- board text added: "GPS"
- board text added: "IS"
